Commit message: refactored ik

File: arm_ik/urdf/Articulated_Arm_Rev2.urdf (robot description, URDF)
Before this commit: robot Articulated_Arm_Rev2, 9 links, 8 joints
Links:
- link chassis_base: geometry collision mesh filename=package://arm_ik/meshes/new_chassis_base.STL; visual mesh filename=package://arm_ik/meshes/new_chassis_base.STL
